File: StepperChecker/_autosave-StepperChecker.sch (KiCad schematic (older format))
At the start: 25 parts, among them J1 PJ-202AH, J12 Terminal, J2 Terminal, J3 FEATHER_A, J4 Molex SL, J5 JST-XH, J6 Dupont, J7 Terminal, J8 FEATHER_B, SW1 BTN_FWD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

Commit message: Add Recom and jumpers
Parts:
- U2: footprint CONV_R-78E5.0-1.0 -> R-78E5.0-1:CONV_R-78E5.0-1.0
Changed lines of the file:
@@
 F 0 "U2" H 2100 3267 50  0000 C CNN
 F 1 "R-78E5.0-1.0" H 2100 3176 50  0000 C CNN
-F 2 "CONV_R-78E5.0-1.0" H 2100 2900 50  0001 L BNN
+F 2 "R-78E5.0-1:CONV_R-78E5.0-1.0" H 2100 2900 50  0001 L BNN
 F 3 "" H 2100 2900 50  0001 L BNN
 F 4 "10.40mm" H 2100 2900 50  0001 L BNN "MAXIMUM_PACKAGE_HEIGHT"
