File: StepperChecker/StepperChecker.sch (KiCad schematic (older format))
At the start: 25 parts, among them J1 PJ-202AH, J12 Terminal, J2 Terminal, J3 FEATHER_A, J4 Molex SL, J5 JST-XH, J6 Dupont, J7 Terminal, J8 FEATHER_B, SW1 BTN_FWD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

Commit message: Minor board tweaks
Parts:
- JP2: value SolderJumper_2_Bridged -> SolderJumper_2_Open; footprint Jumper:SolderJumper-2_P1.3mm_Bridged_RoundedPad1.0x1.5mm -> Jumper:SolderJumper-2_P1.3mm_Open_RoundedPad1.0x1.5mm; symbol Jumper:SolderJumper_2_Bridged -> Jumper:SolderJumper_2_Open
Connections:
- net 5V: no longer VR1.3
- net 3.3V: now reaches J3.2 (Pin_2), U3.2 (3v3)
- net 3.3V: now also VR1.3
Changed lines of the file:
@@
 $EndComp
 Text GLabel 4000 4700 2    31   Input ~ 0
-5V
+3.3V
 $Comp
 L power:GND #PWR05
@@
 	5650 4100 6050 4100
 Wire Wire Line
-	5650 4200 6050 4200
+	5650 4200 5850 4200
 Wire Wire Line
 	6050 4300 5650 4300
@@
 	2700 3100 2950 3100
 $Comp
-L Jumper:SolderJumper_2_Bridged JP2
+L Jumper:SolderJumper_2_Open JP2
 U 1 1 6069EE65
 P 8650 4650
 F 0 "JP2" H 8650 4855 50  0000 C CNN
-F 1 "SolderJumper_2_Bridged" H 8650 4764 50  0000 C CNN
-F 2 "Jumper:SolderJumper-2_P1.3mm_Bridged_RoundedPad1.0x1.5mm" H 8650 4650 50  0001 C CNN
+F 1 "SolderJumper_2_Open" H 8650 4764 50  0000 C CNN
+F 2 "Jumper:SolderJumper-2_P1.3mm_Open_RoundedPad1.0x1.5mm" H 8650 4650 50  0001 C CNN
 F 3 "~" H 8650 4650 50  0001 C CNN
 	1    8650 4650
@@
 Wire Notes Line
 	1000 3450 3400 3450
+Text GLabel 5300 4150 0    31   Input ~ 0
+3.3V
+Wire Wire Line
+	5300 4150 5850 4150
+Wire Wire Line
+	5850 4150 5850 4200
+Connection ~ 5850 4200
+Wire Wire Line
+	5850 4200 6050 4200
 $EndSCHEMATC
